File: KiCAD/DiceDIP_UpperPart/DiceDIP_UpperPart.kicad_pcb (KiCad board)
At the start: 2 copper layers, 40 x 40 mm, 36 parts, among them J1 Conn_01x03, J3 Conn_01x03, J4 Conn_01x06, J5 Conn_01x06, Q1 BC547, SW1 SW_Push, SW2 SW_Push, U1 4029, U2 4093

Commit message: routing upper side done
Parts:
- removed BT1, BT2: Battery_Cell, blinkyparts:BatteryHolder_CR2032_schwarz
- removed C1, C2: 100nF, blinkyparts:C_Disc_D5.0mm_W2.5mm_P5.00mm_handsoldering
- removed C3: 47uF, Capacitor_THT:CP_Radial_D5.0mm_P2.50mm
- removed C4: C, blinkyparts:C_Disc_D5.0mm_W2.5mm_P5.00mm_handsoldering
- removed D1, D10, D9: BAW76, Diode_THT:D_DO-35_SOD27_P7.62mm_Horizontal
- removed D11: 1N4007, Diode_THT:D_DO-41_SOD81_P10.16mm_Horizontal
- removed J1: Conn_01x03, Connector_PinHeader_2.54mm:PinHeader_1x03_P2.54mm_Vertical
- removed J4: Conn_01x06, Connector_PinHeader_2.54mm:PinHeader_1x06_P2.54mm_Vertical
- removed Q1: BC547, Package_TO_SOT_THT:TO-92_HandSolder
- removed R1, R4: 2k2, blinkyparts:R_Axial_DIN0207_L6.3mm_D2.5mm_P7.62mm_Horizontal_handsoldering
- removed R10: R, blinkyparts:R_Axial_DIN0207_L6.3mm_D2.5mm_P7.62mm_Horizontal_handsoldering
- removed R2: 2M2, blinkyparts:R_Axial_DIN0207_L6.3mm_D2.5mm_P7.62mm_Horizontal_handsoldering
- removed R3: 1M, blinkyparts:R_Axial_DIN0207_L6.3mm_D2.5mm_P7.62mm_Horizontal_handsoldering
- removed R5: 120k, blinkyparts:R_Axial_DIN0207_L6.3mm_D2.5mm_P7.62mm_Horizontal_handsoldering
- removed U1: 4029, Package_DIP:DIP-16_W7.62mm_LongPads
- removed U2: 4093, Package_DIP:DIP-14_W7.62mm_LongPads
- J3, J5, R6, R7, R8, R9, SW2: moved to B.Cu
- SW1: moved to F.Cu
- moved D7 94.3 mm to (134.7, 111.0)
- moved D3 91.8 mm to (134.7, 95.0)
- moved D4 90.3 mm to (102.7, 111.0)
- moved SW1 81.9 mm to (116.8, 107.2), turned to 0 degrees
- moved D2 78.4 mm to (102.7, 95.0)
- moved D5 75.7 mm to (134.7, 79.0)
- moved D8 75.7 mm to (118.7, 95.0)
- moved J3 67.1 mm to (111.0, 107.0), turned to 180 degrees
- moved SW2 64.6 mm to (121.3, 89.0), turned to 180 degrees
- moved D6 57.7 mm to (102.7, 79.0)
- moved J5 57.1 mm to (114.0, 78.0), turned to -90 degrees
- moved R7 49.9 mm to (101.8, 102.4)
- moved R6 48.4 mm to (111.0, 90.6), turned to 90 degrees
- moved R8 41.6 mm to (114.2, 93.8), turned to -90 degrees
- moved R9 35.4 mm to (114.2, 90.6), turned to 90 degrees
Routing:
- net Net-(D5-K): track 0.00 -> 83.3 mm
- net Net-(D6-K): track 0.00 -> 74.5 mm, vias 0 -> 1
- net Net-(D4-K): track 0.00 -> 74.2 mm, vias 0 -> 3
- net Net-(D2-K): track 0.00 -> 73.2 mm
- net Net-(J5-Pin_5): track 0.00 -> 53.3 mm
- net Net-(J3-Pin_1): track 0.00 -> 49.5 mm
- net Net-(D3-K): track 0.00 -> 42.0 mm
- net Net-(J5-Pin_6): track 0.00 -> 38.2 mm
- net Net-(J3-Pin_2): track 0.00 -> 29.0 mm
- net Net-(D6-A): track 0.00 -> 18.5 mm
- net Net-(D4-A): track 0.00 -> 16.3 mm
- net Net-(J5-Pin_4): track 0.00 -> 12.7 mm
- net Net-(J3-Pin_3): track 0.00 -> 12.0 mm
- net Net-(D8-A): track 0.00 -> 9.99 mm, vias 0 -> 2
- net Net-(D2-A): track 0.00 -> 7.55 mm
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- added copper zone on B.Cu, net (none)
- added copper zone on F.Cu, net (none)

Commit message: minor changes
Parts:
- moved J3 19.0 mm to (130.0, 106.0)
- moved R7 17.8 mm to (119.6, 102.5)
- moved R9 10.7 mm to (119.9, 81.5), turned to 180 degrees
- moved SW2 8.86 mm to (114.8, 95.0)
- moved R8 8.00 mm to (117.5, 86.5), turned to 0 degrees
- moved R6 6.50 mm to (117.4, 89.8), turned to 0 degrees
- moved J5 4.00 mm to (110.0, 78.0)
Routing:
- net Net-(J3-Pin_1): track 49.5 -> 19.8 mm
- net Net-(J3-Pin_2): track 29.0 -> 7.18 mm
- net Net-(J3-Pin_3): track 12.0 -> 28.3 mm
- net Net-(D2-K): track 73.2 -> 86.1 mm
- net Net-(J5-Pin_4): track 12.7 -> 25.4 mm, vias 0 -> 2
- net Net-(J5-Pin_5): track 53.3 -> 63.3 mm, vias 0 -> 4
- net Net-(D5-K): track 83.3 -> 92.9 mm
- net Net-(D2-A): track 7.55 -> 15.5 mm
- net Net-(D8-A): track 9.99 -> 15.2 mm, vias 2 -> 0
- net Net-(D3-K): track 42.0 -> 46.2 mm
- net Net-(D4-A): track 16.3 -> 20.4 mm
- net Net-(D6-A): track 18.5 -> 15.3 mm
- net Net-(D4-K): track 74.2 -> 75.4 mm, vias 3 -> 2

Commit message: changed some silkscreen and updated gerber-files
Parts:
- added blinkyparts_logo_5mm: G***, blinkyparts:logo_blinkyparts_5mm_F.Mask, F.Cu at (133.2, 100.8)
- added ce-symbol_mask_3mm: G***, blinkyparts:legislation_ce-icon_3mm_F.Mask, B.Cu at (112.9, 104.4)
- added weee-symbol_mask_3mm: G***, blinkyparts:legislation_weee-icon_3mm_F.Mask, B.Cu at (107.4, 104.4)
Other:
- board text added: "DiceDIP UpperPart v2.0"
- board text added: "Product & Design by blinkyparts.com Egerstr. 9, 93057 Rgb"
